File: zmod/zmod.kicad_sch (KiCad schematic)
At the start: 0 parts

Commit message: starting to route zmod diff pairs
Parts:
- added D1, D2: LED, LED_SMD:LED_0603_1608Metric, symbol Device:LED
- added H1, H2, H3, H4, H5, H6: MountingHole_Pad, MountingHole:MountingHole_3.2mm_M3_DIN965_Pad_TopBottom, symbol Mechanical:MountingHole_Pad
- added J2: QTH-020-01-X-D-DP-A, SAMTEC_QTH-020-01-X-D-DP-A, symbol QTH-020-01-X-D-DP-A:QTH-020-01-X-D-DP-A
- added R1, R2: 240, Resistor_SMD:R_0603_1608Metric, symbol Device:R
- added R3: 100, Resistor_SMD:R_0603_1608Metric, symbol Device:R
- added R5: 10k,1%, Resistor_SMD:R_0603_1608Metric, symbol Device:R
Connections:
- new net: D2.2 (A), R2.1
- new net: J2.16, R2.2
- new net: J2.14, R1.2
- new net: D1.2 (A), R1.1
- new net +3V3: J2.40, R5.1
- new net +5V: J2.02
- new net GND: D1.1 (K), D2.1 (K), J2.G1 (GND), J2.G2 (GND), J2.G3 (GND), J2.G4 (GND)
- new net R_GA: J2.04, R5.2
- new net SCL: J2.01
- new net SDA: J2.03
- new net VIO: J2.39
- new net hss0_N: J2.07, J2.08
- new net hss0_P: J2.05, J2.06
- new net hss1_N: J2.11, J2.12
- new net hss1_P: J2.09, J2.10
- new net lvds0_N: J2.19, J2.23
- new net lvds0_P: J2.17, J2.21
- new net lvds1_N: J2.27, J2.31
- new net lvds1_P: J2.25, J2.29
- new net lvds2_N: J2.28, J2.32
- new net lvds2_P: J2.26, J2.30
- new net lvds3_N: J2.20, J2.24
- new net lvds3_P: J2.18, J2.22
- new net lvdsclk_N: J2.35, J2.36
- new net lvdsclk_P: J2.33, J2.34
- new net refclk_N: J2.15, R3.2
- new net refclk_P: J2.13, R3.1
- new net rsvd1: J2.37
- new net rsvd2: J2.38
Other:
- note added: "ZMOD TXR-2 Loopback Board"
- note added: "www.hdlguy.com"
