File: zmod_standard/zmod.kicad_sch (KiCad schematic)
At the start: 13 parts, among them J2 QTH-020-01-X-D-DP-A

Commit message: zmod_standard work
Parts:
- removed J2: QTH-020-01-X-D-DP-A, SAMTEC_QTH-020-01-X-D-DP-A, symbol QTH-020-01-X-D-DP-A:QTH-020-01-X-D-DP-A
- removed R3: 100, Resistor_SMD:R_0603_1608Metric, symbol Device:R
- added J1: QTE-020-01-X-D-A, SAMTEC_QTE-020-01-X-D-A, symbol QTE-020-01-F-D-A:QTE-020-01-X-D-A
Connections:
- net +3V3: now also J1.40 (+3.3V)
- net +5V: now also J1.02 (+5V)
- net GND: now also J1.G1 (GND), J1.G2 (GND), J1.G3 (GND), J1.G4 (GND)
- net R_GA: now also J1.04 (R_GA)
- net led1: now reaches R2.2
- net led1: now also J1.32 (S27)
- net led0: now reaches R1.2
- net led0: now also J1.30 (S25)
- new net d0_N: J1.07 (S2_D0N), J1.11 (S6_D2N)
- new net d0_P: J1.05 (S0_D0P), J1.09 (S4_D2P)
- new net d1_N: J1.08 (S3_D1N), J1.12 (S7_D3N)
- new net d1_P: J1.06 (S1_D1P), J1.10 (S5_D3P)
- new net d4_N: J1.15 (S10_D4N), J1.19 (S14_D6N)
- new net d4_P: J1.13 (S8_D4P), J1.17 (S12_D6P)
- new net d5_N: J1.16 (S11_D5N), J1.20 (S15_D7N)
- new net d5_P: J1.14 (S9_D5P), J1.18 (S13_D7P)
- new net p2c_clk_N: J1.35 (P2C_CLKN), J1.36 (C2P_CLKN)
- new net p2c_clk_P: J1.33 (P2C_CLKP), J1.34 (C2P_CLKP)
- new net s16: J1.21 (S16), J1.23 (S18)
- new net s17: J1.22 (S17), J1.24 (S19)
- new net s20: J1.25 (S20), J1.27 (S22)
- new net s21: J1.26 (S21), J1.28 (S23)
- new net s24: J1.29 (S24), J1.31 (S26)
Other:
- note added: "ZMOD Standard Loopback Board"
- note removed: "ZMOD TXR-2 Loopback Board"
- moved on the sheet: D1, D2, R1, R2, R5

Commit message: organizing local libraries, footprint and symbol
Parts:
- J1: footprint SAMTEC_QTE-020-01-X-D-A -> pedrolib:SAMTEC_QTE-020-01-X-D-A; symbol QTE-020-01-F-D-A:QTE-020-01-X-D-A -> pedrolib:QTE-020-01-X-D-A
Changed lines of the file:
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@@
     (pin "1")
   )
-  (symbol (lib_id "QTE-020-01-F-D-A:QTE-020-01-X-D-A") (at 128.27 95.25 0) (unit 1)
+  (symbol (lib_id "pedrolib:QTE-020-01-X-D-A") (at 128.27 95.25 0) (unit 1)
     (in_bom yes) (on_board yes) (fields_autoplaced)
     (property "Reference" "J1" (id 0) (at 125.095 62.23 0))
     (property "Value" "QTE-020-01-X-D-A" (id 1) (at 125.095 64.77 0))
-    (property "Footprint" "SAMTEC_QTE-020-01-X-D-A" (id 2) (at 109.22 64.77 0)
+    (property "Footprint" "pedrolib:SAMTEC_QTE-020-01-X-D-A" (id 2) (at 109.22 64.77 0)
       (effects (font (size 1.27 1.27)) (justify left bottom) hide)
     )
@@
     )
     (path "/d2960b08-94ac-4444-9a28-848c3a20e1f1"
-      (reference "J1") (unit 1) (value "QTE-020-01-X-D-A") (footprint "SAMTEC_QTE-020-01-X-D-A")
+      (reference "J1") (unit 1) (value "QTE-020-01-X-D-A") (footprint "pedrolib:SAMTEC_QTE-020-01-X-D-A")
     )
     (path "/ff644ff7-2624-41c7-a7cc-9f9e7511816f"
