File: zmod_txr-2/zmod.kicad_pcb (KiCad board)
At the start: 6 copper layers, 50 x 70 mm, 13 parts, among them J2 QTH-020-01-X-D-DP-A

Commit message: added M.2-m connector to the design for a sata ssd
Parts:
- removed R3: 100, Resistor_SMD:R_0603_1608Metric
- added J1: MDT420M02001, 1-2199230-5:TE_1-2199230-5, F.Cu at (128.0, 75.3)
- moved D1 21.7 mm to (106.0, 80.2)
- moved D2 21.7 mm to (103.0, 80.2)
- moved R1 21.7 mm to (106.0, 75.6)
- moved R2 21.7 mm to (103.0, 75.6)
Connections:
- J2 pad 05: /hss0_P -> unconnected-(J2-Pad05)
- J2 pad 06: /hss0_P -> unconnected-(J2-Pad06)
- J2 pad 07: /hss0_N -> unconnected-(J2-Pad07)
- J2 pad 08: /hss0_N -> unconnected-(J2-Pad08)
- J2 pad 09: /hss1_P -> unconnected-(J2-Pad09)
- J2 pad 10: /hss1_P -> unconnected-(J2-Pad10)
- J2 pad 11: /hss1_N -> unconnected-(J2-Pad11)
- J2 pad 12: /hss1_N -> unconnected-(J2-Pad12)
Routing:
- net /hss1_N: track 353.6 -> 0.00 mm, vias 12 -> 0
- net /hss1_P: track 353.5 -> 0.00 mm, vias 12 -> 0
- net Net-(J2-Pad14): track 52.9 -> 0.00 mm, vias 2 -> 0
- net Net-(J2-Pad16): track 52.8 -> 0.00 mm, vias 2 -> 0
- net /lvdsclk_P: track 27.2 -> 0.00 mm
- net /lvdsclk_N: track 24.2 -> 0.00 mm
- net /lvds1_P: track 15.5 -> 0.00 mm, vias 2 -> 0
- net /lvds1_N: track 12.8 -> 0.00 mm, vias 2 -> 0
- net /lvds0_P: track 12.1 -> 0.00 mm, vias 2 -> 0
- net /lvds0_N: track 10.8 -> 0.00 mm, vias 2 -> 0
- net /lvds2_P: track 8.56 -> 0.00 mm, vias 2 -> 0
- net /refclk_N: track 8.27 -> 0.00 mm
- net /refclk_P: track 8.25 -> 0.00 mm
- net /lvds3_P: track 7.34 -> 0.00 mm, vias 2 -> 0
- net /lvds2_N: track 7.26 -> 0.00 mm, vias 2 -> 0
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
Commit message: organizing local libraries, footprint and symbol
Parts:
- J1: footprint 1-2199230-5:TE_1-2199230-5 -> pedrolib:TE_1-2199230-5
- J2: footprint QTH:SAMTEC_QTH-020-01-X-D-DP-A -> pedrolib:SAMTEC_QTH-020-01-X-D-DP-A
