File: zmod_txr-2/zmod.kicad_pcb (KiCad board)
At the start: 6 copper layers, 50 x 70 mm, 13 parts, among them J1 MDT420M02001, J2 QTH-020-01-X-D-DP-A

Commit message: working on M.2 ZMOD board
Parts:
- removed D1, D2: LED, LED_SMD:LED_0603_1608Metric
- removed R1, R2: 240, Resistor_SMD:R_0603_1608Metric
- added C1: C, Capacitor_SMD:C_0603_1608Metric, F.Cu at (130.0, 63.9)
- added C2: C, Capacitor_SMD:C_0603_1608Metric, F.Cu at (123.0, 63.9)
- added C3: C, Capacitor_SMD:C_0603_1608Metric, F.Cu at (132.0, 63.9)
- added C4: C, Capacitor_SMD:C_0603_1608Metric, F.Cu at (125.0, 63.9)
- added D3: LED, LED_SMD:LED_0603_1608Metric, F.Cu at (105.0, 106.0)
- added R3: 240, Resistor_SMD:R_0603_1608Metric, F.Cu at (105.0, 101.0)
- added U1: SN74LVC1T45DBV, Package_TO_SOT_SMD:SOT-23-6, F.Cu at (107.1, 78.0)
Connections:
- J1 pad 10: unconnected-(J1-Pad10) -> Net-(J1-Pad10)
- J1 pad 29: unconnected-(J1-Pad29) -> /gtr1_rxn
- J1 pad 31: unconnected-(J1-Pad31) -> /gtr1_rxp
- J1 pad 35: unconnected-(J1-Pad35) -> Net-(J1-Pad35)
- J1 pad 37: unconnected-(J1-Pad37) -> Net-(J1-Pad37)
- J1 pad 41: unconnected-(J1-Pad41) -> /gtr0_rxn
- J1 pad 43: unconnected-(J1-Pad43) -> /gtr0_rxp
- J1 pad 47: unconnected-(J1-Pad47) -> Net-(J1-Pad47)
- J1 pad 49: unconnected-(J1-Pad49) -> Net-(J1-Pad49)
- J1 pad 50: unconnected-(J1-Pad50) -> Net-(J1-Pad50)
- J1 pad 53: /refclk_N -> unconnected-(J1-Pad53)
- J1 pad 55: /refclk_P -> unconnected-(J1-Pad55)
- J2 pad 05: unconnected-(J2-Pad05) -> /gtr0_rxp
- J2 pad 06: unconnected-(J2-Pad06) -> /gtr0_txp
- J2 pad 07: unconnected-(J2-Pad07) -> /gtr0_rxn
- J2 pad 08: unconnected-(J2-Pad08) -> /gtr0_txn
- J2 pad 09: unconnected-(J2-Pad09) -> /gtr1_rxp
- J2 pad 10: unconnected-(J2-Pad10) -> /gtr1_txp
- J2 pad 11: unconnected-(J2-Pad11) -> /gtr1_rxn
- J2 pad 12: unconnected-(J2-Pad12) -> /gtr1_txn
- J2 pad 13: /refclk_P -> /gtrclk0_p
- J2 pad 14: Net-(J2-Pad14) -> /lvds3_P
- J2 pad 15: /refclk_N -> /gtrclk0_n
- J2 pad 16: Net-(J2-Pad16) -> /lvds3_N
- J2 pad 22: /lvds3_P -> /lvds2_P
- J2 pad 24: /lvds3_N -> /lvds2_N
- J2 pad 30: /lvds2_P -> Net-(J2-Pad30)
- J2 pad 32: /lvds2_N -> unconnected-(J2-Pad32)
- J2 pad 39: /VIO -> +1V8
Routing:
- net Net-(D2-Pad2): track 2.97 -> 0.00 mm
- net Net-(D1-Pad2): track 2.97 -> 0.00 mm
- net GND: track 9.25 -> 6.59 mm, vias 10 -> 8
