File: microzed_carrier/microzed_carrier.kicad_pcb (KiCad board)
At the start: 2 copper layers, 82.5 x 101.6 mm, 15 parts, among them J1 Jack-DC, P1 61083-101400LF, P2 61083-101400LF

Commit message: added CUI barrel connector for 5V power
Parts:
- J1: value Jack-DC -> PJ-002AH-SMT-TR; footprint Connector_BarrelJack:BarrelJack_CLIFF_FC681465S_SMT_Horizontal -> pedrolib:CUI_PJ-002AH-SMT-TR
- moved J1 8.34 mm to (174.0, 62.0)
Connections:
- J1 pad 3: (no net) -> unconnected-(J1-Pad3)
Changed lines of the file:
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@@
   (net 150 "unconnected-(H3-Pad1)")
   (net 151 "unconnected-(H4-Pad1)")
-  (net 152 "unconnected-(J1-Pad1)")
+  (net 152 "Net-(J1-Pad1A)")
   (net 153 "unconnected-(J1-Pad2)")
   (net 154 "unconnected-(D1-Pad1)")
@@
   (net 168 "unconnected-(R4-Pad1)")
   (net 169 "unconnected-(R4-Pad2)")
+  (net 170 "unconnected-(J1-Pad3)")
   (footprint "pedrolib:FCI_61083-101400LF" locked (layer "F.Cu")
     (at 149.23135 101.6 -90)
@@
     (property "Sheetname" "")
     (attr through_hole)
-    (fp_text reference "P1" (at -19.895525 -5.019055 -90) (layer "F.SilkS")
+    (fp_text reference "P1" (at -24.6 0.23135) (layer "F.SilkS")
       (effects (font (size 1.003551 1.003551) (thickness 0.15)))
     )
@@
     (property "Sheetname" "")
     (attr through_hole)
-    (fp_text reference "P2" (at -19.895525 -5.019055 -90) (layer "F.SilkS")
+    (fp_text reference "P2" (at -24.6 -0.23135) (layer "F.SilkS")
       (effects (font (size 1.003551 1.003551) (thickness 0.15)))
     )
@@
       (net 148 "unconnected-(H1-Pad1)") (pinfunction "1") (pintype "input"))
   )
+  (footprint "pedrolib:CUI_PJ-002AH-SMT-TR" (layer "F.Cu")
+    (at 174 62 -90)
+    (property "MANUFACTURER" "CUI INC")
+    (property "STANDARD" "Manufacturer recommendations")
+    (property "Sheetfile" "microzed_carrier.kicad_sch")
+    (property "Sheetname" "")
+    (attr through_hole)
+    (fp_text reference "J1" (at 7 6 180) (layer "F.SilkS")
+      (effects (font (size 1.000976 1.000976) (thickness 0.15)))
+    )
+    (fp_text value "PJ-002AH-SMT-TR" (at 0.6062 14.3119 90) (layer "F.Fab")
+      (effects (font (size 1.00189 1.00189) (thickness 0.15)))
+    )
+    (fp_line (start -11.1 10.2) (end -7.7 10.2) (layer "F.SilkS") (width 0.127))
+    (fp_line (start 1.6 10.2) (end 3.7 10.2) (layer "F.SilkS") (width 0.127))
+    (fp_line (start -1.6 1.2) (end -4.5 1.2) (layer "F.SilkS") (width 0.127))
+    (fp_line (start 2.65 1.2) (end 1.6 1.2) (layer "F.SilkS") (width 0.127))
+    (fp_line (start -7.7 1.2) (end -11.1 1.2) (layer "F.SilkS") (width 0.127))
+    (fp_line (start 3.15 7) (end 3.15 3.55) (layer "F.SilkS") (width 0.127))
+    (fp_line (start 3.15 3.55) (end 2.65 3.55) (layer "F.SilkS") (width 0.127))
+    (fp_line (start -11.1 1.2) (end -11.1 10.2) (layer "F.SilkS") (width 0.127))
+    (fp_line (start 2.65 3.55) (end 2.65 1.2) (layer "F.SilkS") (width 0.127))
+    (fp_line (start 3.7 7) (end 3.15 7) (layer "F.SilkS") (width 0.127))
+    (fp_line (start 3.7 10.2) (end 3.7 7) (layer "F.SilkS") (width 0.127))
+    (fp_line (start -4.5 10.2) (end -1.6 10.2) (layer "F.SilkS") (width 0.127))
+    (fp_circle (center 0 -1.99) (end 0.2 -1.99) (layer "F.SilkS") (width 0.4) (fill none))
+    (fp_line (start 3.95 10.45) (end 1.65 10.45) (layer "F.CrtYd") (width 0.05))
+    (fp_line (start -4.45 -1.45) (end -4.45 0.95) (layer "F.CrtYd") (width 0.05))
+    (fp_line (start 1.65 12.85) (end -1.65 12.85) (layer "F.CrtYd") (width 0.05))
+    (fp_line (start 1.65 10.45) (end 1.65 12.85) (layer "F.CrtYd") (width 0.05))
+    (fp_line (start 1.65 -1.45) (end 1.65 0.95) (layer "F.CrtYd") (width 0.05))
+    (fp_line (start -7.75 0.95) (end -7.75 -1.45) (layer "F.CrtYd") (width 0.05))
+    (fp_line (start -4.45 0.95) (end -1.65 0.95) (layer "F.CrtYd") (width 0.05))
+    (fp_line (start -1.65 -1.45) (end 1.65 -1.45) (layer "F.CrtYd") (width 0.05))
+    (fp_line (start -1.65 0.95) (end -1.65 -1.45) (layer "F.CrtYd") (width 0.05))
+    (fp_line (start 1.65 0.95) (end 3.95 0.95) (layer "F.CrtYd") (width 0.05))
+    (fp_line (start -7.75 10.45) (end -11.35 10.45) (layer "F.CrtYd") (width 0.05))
+    (fp_line (start -11.35 10.45) (end -11.35 0.95) (layer "F.CrtYd") (width 0.05))
+    (fp_line (start -7.75 12.85) (end -7.75 10.45) (layer "F.CrtYd") (width 0.05))
+    (fp_line (start -1.65 10.45) (end -4.45 10.45) (layer "F.CrtYd") (width 0.05))
+    (fp_line (start -11.35 0.95) (end -7.75 0.95) (layer "F.CrtYd") (width 0.05))
+    (fp_line (start -4.45 12.85) (end -7.75 12.85) (layer "F.CrtYd") (width 0.05))
+    (fp_line (start -1.65 12.85) (end -1.65 10.45) (layer "F.CrtYd") (width 0.05))
+    (fp_line (start -4.45 10.45) (end -4.45 12.85) (layer "F.CrtYd") (width 0.05))
+    (fp_line (start 3.95 0.95) (end 3.95 10.45) (layer "F.CrtYd") (width 0.05))
+    (fp_line (start -7.75 -1.45) (end -4.45 -1.45) (layer "F.CrtYd") (width 0.05))
+    (fp_line (start -11.1 1.2) (end -11.1 10.2) (layer "F.Fab") (width 0.127))
+    (fp_line (start 3.7 10.2) (end 3.7 1.2) (layer "F.Fab") (width 0.127))
+    (fp_line (start 3.7 1.2) (end -11.1 1.2) (layer "F.Fab") (width 0.127))
+    (fp_line (start -11.1 10.2) (end 3.7 10.2) (layer "F.Fab") (width 0.127))
+    (pad "" np_thru_hole circle (at -6.1 5.7 270) (size 1.7 1.7) (drill 1.7) (layers *.Cu *.Mask))
+    (pad "" np_thru_hole circle (at -1.6 5.7 270) (size 1.8 1.8) (drill 1.8) (layers *.Cu *.Mask))
+    (pad "1A" smd rect (at 0 0 270) (size 2.8 2.4) (layers "F.Cu" "F.Paste" "F.Mask")
+      (net 152 "Net-(J1-Pad1A)") (pintype "passive"))
+    (pad "1B" smd rect (at -6.1 0 270) (size 2.8 2.4) (layers "F.Cu" "F.Paste" "F.Mask")
+      (net 152 "Net-(J1-Pad1A)") (pintype "passive"))
+    (pad "2" smd rect (at -6.1 11.4 270) (size 2.8 2.4) (layers "F.Cu" "F.Paste" "F.Mask")
+      (net 153 "unconnected-(J1-Pad2)") (pintype "passive"))
+    (pad "3" smd rect (at 0 11.4 270) (size 2.8 2.4) (layers "F.Cu" "F.Paste" "F.Mask")
+      (net 170 "unconnected-(J1-Pad3)") (pintype "passive"))
+    (model "/home/pedro/github/my_kicad/libs/step/CUI_DEVICES_PJ-002AH-SMT-TR.step"
+      (offset (xyz -11 -5.62 0))
+      (scale (xyz 1 1 1))
+      (rotate (xyz -90 0 90))
+    )
+  )
   (footprint "LED_SMD:LED_0603_1608Metric" (layer "F.Cu")
     (at 121.525 134.105)
@@
       (offset (xyz 0 0 0))
       (scale (xyz 1 1 1))
-      (rotate (xyz 0 0 0))
-    )
-  )
-  (footprint "Connector_BarrelJack:BarrelJack_CLIFF_FC681465S_SMT_Horizontal" (layer "F.Cu")
-    (at 167.275 57.075 -90)
-    (descr "Surface-mount DC Barrel Jack, https://www.cliffuk.co.uk/products/dcconnectors/FC681465S.pdf")
-    (tags "Power Jack SMT")
-    (property "Sheetfile" "microzed_carrier.kicad_sch")
-    (property "Sheetname" "")
-    (attr smd)
-    (fp_text reference "J1" (at -6.5 6.5 90) (layer "F.SilkS")
-      (effects (font (size 1 1) (thickness 0.15)))
-    )
-    (fp_text value "Jack-DC" (at -0.5 8.5 90) (layer "F.Fab")
-      (effects (font (size 1 1) (thickness 0.15)))
-    )
-    (fp_text user "${REFERENCE}" (at -0.5 0.5 90) (layer "F.Fab")
-      (effects (font (size 1 1) (thickness 0.15)))
-    )
-    (fp_line (start -1.5 4.56) (end 1.5 4.56) (layer "F.SilkS") (width 0.12))
-    (fp_line (start -4.26 -7.26) (end -4.26 -5.36) (layer "F.SilkS") (width 0.12))
-    (fp_line (start 4.5 4.56) (end 6.81 4.56) (layer "F.SilkS") (width 0.12))
-    (fp_line (start -4.8 -3) (end 0 -3) (layer "F.SilkS") (width 0.12))
-    (fp_line (start -2.92 -7.26) (end -4.26 -7.26) (layer "F.SilkS") (width 0.12))
-    (fp_line (start -8.11 4.56) (end -8.11 -4.56) (layer "F.SilkS") (width 0.12))
-    (fp_line (start -1.5 -4.56) (end 1.5 -4.56) (layer "F.SilkS") (width 0.12))
-    (fp_line (start -4.8 4.56) (end -4.8 -4.56) (layer "F.SilkS") (width 0.12))
-    (fp_line (start -8.11 -4.56) (end -4.5 -4.56) (layer "F.SilkS") (width 0.12))
-    (fp_line (start -8.11 4.56) (end -4.5 4.56) (layer "F.SilkS") (width 0.12))
-    (fp_line (start -4.8 3) (end 0 3) (layer "F.SilkS") (width 0.12))
-    (fp_line (start 6.81 4.56) (end 6.81 -4.56) (layer "F.SilkS") (width 0.12))
-    (fp_line (start 4.5 -4.56) (end 6.81 -4.56) (layer "F.SilkS") (width 0.12))
-    (fp_arc (start 0 -3) (mid 3 0) (end 0 3) (layer "F.SilkS") (width 0.12))
-    (fp_line (start -8.5 7.5) (end 7.2 7.5) (layer "F.CrtYd") (width 0.05))
-    (fp_line (start -8.5 7.5) (end -8.5 -7.5) (layer "F.CrtYd") (width 0.05))
-    (fp_line (start 7.2 7.5) (end 7.2 -7.5) (layer "F.CrtYd") (width 0.05))
-    (fp_line (start -8.5 -7.5) (end 7.2 -7.5) (layer "F.CrtYd") (width 0.05))
-    (fp_line (start -8 4.45) (end -8 -4.45) (layer "F.Fab") (width 0.1))
-    (fp_line (start -4 -4.45) (end -3 -3.5) (layer "F.Fab") (width 0.1))
-    (fp_line (start -8 -4.45) (end -4 -4.45) (layer "F.Fab") (width 0.1))
-    (fp_line (start -3 -3.5) (end -2 -4.45) (layer "F.Fab") (width 0.1))
-    (fp_line (start 6.7 4.45) (end 6.7 -4.45) (layer "F.Fab") (width 0.1))
-    (fp_line (start -8 4.45) (end 6.7 4.45) (layer "F.Fab") (width 0.1))
-    (fp_line (start -2 -4.45) (end 6.7 -4.45) (layer "F.Fab") (width 0.1))
-    (pad "" np_thru_hole oval (at -2.9 0) (size 2 1.5) (drill oval 2 1.5) (layers *.Cu *.Mask))
-    (pad "" np_thru_hole circle (at 1.5 0) (size 2 2) (drill 2) (layers *.Cu *.Mask))
-    (pad "1" smd rect (at -3 -5.5) (size 3 2) (layers "F.Cu" "F.Paste" "F.Mask")
-      (net 152 "unconnected-(J1-Pad1)") (pintype "passive"))
-    (pad "1" smd rect (at 3 -5.5) (size 3 2) (layers "F.Cu" "F.Paste" "F.Mask")
-      (net 152 "unconnected-(J1-Pad1)") (pintype "passive"))
-    (pad "2" smd rect (at 3 5.5) (size 3 2) (layers "F.Cu" "F.Paste" "F.Mask")
-      (net 153 "unconnected-(J1-Pad2)") (pintype "passive"))
-    (pad "3" smd rect (at -3 5.5) (size 3 2) (layers "F.Cu" "F.Paste" "F.Mask"))
-    (model "${KICAD6_3DMODEL_DIR}/Connector_BarrelJack.3dshapes/BarrelJack_CLIFF_FC681465S_SMT_Horizontal.wrl"
-      (offset (xyz 0 0 0))
-      (scale (xyz 1 1 1))
