File: microzed_carrier/microzed_carrier.kicad_sch (KiCad schematic)
At the start: 15 parts, among them J1 Jack-DC, P1 61083-101400LF, P2 61083-101400LF

Commit message: added CUI barrel connector for 5V power
Parts:
- removed J1: Jack-DC, Connector_BarrelJack:BarrelJack_CLIFF_FC681465S_SMT_Horizontal, symbol Connector:Jack-DC
- added J1: PJ-002AH-SMT-TR, pedrolib:CUI_PJ-002AH-SMT-TR, symbol pedrolib:PJ-002AH-SMT-TR
Connections:
- new net: J1.1A, J1.1B
Changed lines of the file:
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@@
     (pin "1")
+  )
+  (symbol (lib_id "pedrolib:PJ-002AH-SMT-TR") (at 85.09 182.88 0) (unit 1)
+    (in_bom yes) (on_board yes) (fields_autoplaced)
+    (property "Reference" "J1" (id 0) (at 81.8515 172.72 0))
+    (property "Value" "PJ-002AH-SMT-TR" (id 1) (at 81.8515 175.26 0))
+    (property "Footprint" "pedrolib:CUI_PJ-002AH-SMT-TR" (id 2) (at 85.09 182.88 0)
+      (effects (font (size 1.27 1.27)) (justify left bottom) hide)
+    )
+    (property "Datasheet" "" (id 3) (at 85.09 182.88 0)
+      (effects (font (size 1.27 1.27)) (justify left bottom) hide)
+    )
+    (property "STANDARD" "Manufacturer recommendations" (id 4) (at 85.09 182.88 0)
+      (effects (font (size 1.27 1.27)) (justify left bottom) hide)
+    )
+    (property "MANUFACTURER" "CUI INC" (id 5) (at 85.09 182.88 0)
+      (effects (font (size 1.27 1.27)) (justify left bottom) hide)
+    )
+    (pin "1A")
+    (pin "1B")
+    (pin "2")
+    (pin "3")
   )
   (symbol (lib_id "power:GND") (at 212.09 158.75 0) (unit 1)
@@
     )
     (pin "1")
-  )
-  (symbol (lib_id "Connector:Jack-DC") (at 72.39 185.42 0) (unit 1)
-    (in_bom yes) (on_board yes) (fields_autoplaced)
-    (property "Reference" "J1" (id 0) (at 72.39 176.53 0))
-    (property "Value" "Jack-DC" (id 1) (at 72.39 179.07 0))
-    (property "Footprint" "Connector_BarrelJack:BarrelJack_CLIFF_FC681465S_SMT_Horizontal" (id 2) (at 73.66 186.436 0)
-      (effects (font (size 1.27 1.27)) hide)
-    )
-    (property "Datasheet" "~" (id 3) (at 73.66 186.436 0)
-      (effects (font (size 1.27 1.27)) hide)
-    )
-    (pin "1")
-    (pin "2")
   )
   (symbol (lib_id "pedrolib:microzed_mount_hole") (at 33.02 173.99 270) (unit 1)
@@
       (reference "H4") (unit 1) (value "microzed_mount_hole") (footprint "MountingHole:MountingHole_3.2mm_M3_Pad")
     )
-    (path "/9fc6d450-5606-44ce-83b3-99d14ffbb0fb"
-      (reference "J1") (unit 1) (value "Jack-DC") (footprint "Connector_BarrelJack:BarrelJack_CLIFF_FC681465S_SMT_Horizontal")
+    (path "/4d2c55a0-0161-415b-822d-6908b35f349b"
+      (reference "J1") (unit 1) (value "PJ-002AH-SMT-TR") (footprint "pedrolib:CUI_PJ-002AH-SMT-TR")
     )
     (path "/2f0771ac-785e-49cd-b5db-9060c3cbc2f1"
