File: kria_carrier/kria_carrier.kicad_sch (KiCad schematic)
At the start: 2 parts, among them J1 ADM6-60-01.5-L-4-2-A-TR, J2 ADM6-60-01.5-L-4-2-A-TR

Commit message: library paths are messed up
Parts:
- added H1, H2, H3, H4: Kria_mounting_hole, MountingHole:MountingHole_4.5mm_Pad, symbol pedrolib:Kria_mounting_hole
- added H5, H6, H7, H8: standoff_hole, MountingHole:MountingHole_3.5mm_Pad, symbol pedrolib:standoff_hole
- added unit 2 of J1
- added unit 2 of J2
Other:
- note added: "Corner standoff holes"
- note added: "Kria mounting holes"
- moved on the sheet: J2A

Commit message: straitened out the pedrolib path for the kria carrier at least
Parts:
- J1: symbol pedrolib:ADM6-60-01.5-L-4-2-A-TR -> pedrolib:kria_conn_1
- J2: symbol pedrolib:ADM6-60-01.5-L-4-2-A-TR -> pedrolib:kria_conn_2
Changed lines of the file:
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@@
     (pin "1")
   )
-  (symbol (lib_id "pedrolib:ADM6-60-01.5-L-4-2-A-TR") (at 109.22 293.37 0) (unit 1)
+  (symbol (lib_id "pedrolib:kria_conn_2") (at 109.22 293.37 0) (unit 1)
     (in_bom yes) (on_board yes) (fields_autoplaced)
     (property "Reference" "J2" (id 0) (at 109.22 212.09 0))
@@
     (pin "1")
   )
-  (symbol (lib_id "pedrolib:ADM6-60-01.5-L-4-2-A-TR") (at 160.02 297.18 0) (unit 2)
+  (symbol (lib_id "pedrolib:kria_conn_2") (at 160.02 297.18 0) (unit 2)
     (in_bom yes) (on_board yes) (fields_autoplaced)
     (property "Reference" "J2" (id 0) (at 160.02 215.9 0))
@@
     (pin "D60")
   )
-  (symbol (lib_id "pedrolib:ADM6-60-01.5-L-4-2-A-TR") (at 110.49 101.6 0) (unit 1)
+  (symbol (lib_id "pedrolib:kria_conn_1") (at 110.49 101.6 0) (unit 1)
     (in_bom yes) (on_board yes) (fields_autoplaced)
     (property "Reference" "J1" (id 0) (at 110.49 20.32 0))
@@
     (pin "D60")
   )
-  (symbol (lib_id "pedrolib:ADM6-60-01.5-L-4-2-A-TR") (at 153.67 99.06 0) (unit 2)
+  (symbol (lib_id "pedrolib:kria_conn_1") (at 153.67 99.06 0) (unit 2)
     (in_bom yes) (on_board yes) (fields_autoplaced)
     (property "Reference" "J1" (id 0) (at 153.67 17.78 0))

Commit message: working on the power connections to the kria connectors. That connector will be tight to escape.
Connections:
- net GND: now reaches H7.1
- net GND: now also H1.1, H2.1, H3.1, H4.1, H5.1, H6.1, H8.1, J1.A02 (GND), J1.A05 (GND), J1.A08 (GND), J1.A11 (GND), J1.A14 (GND), J1.A18 (GND), J1.A21 (GND), J1.A26 (GND), J1.A33 (GND), J1.A37 (GND), J1.A41 (GND), J1.A45 (GND), J1.A46 (GND), J1.A49 (GND), J1.A50 (GND), J1.A53 (GND), J1.A54 (GND), J1.A57 (GND), J1.A58 (GND), J1.B03 (GND), J1.B06 (GND), J1.B08 (GND), J1.B12 (GND), J1.B15 (GND), J1.B19 (GND), J1.B23 (GND), J1.B27 (GND), J1.B31 (GND), J1.B35 (GND), J1.B39 (GND), J1.B43 (GND), J1.B47 (GND), J1.B48 (GND), J1.B51 (GND), J1.B52 (GND), J1.B55 (GND), J1.B56 (GND), J1.B59 (GND), J1.C01 (GND), J1.C05 (GND), J1.C08 (GND), J1.C11 (GND), J1.C14 (GND), J1.C17 (GND), J1.C21 (GND), J1.C25 (GND), J1.C29 (GND), J1.C33 (GND), J1.C37 (GND), J1.C41 (GND), J1.C46 (GND), J1.C49 (GND), J1.C50 (GND), J1.C53 (GND), J1.C54 (GND), J1.C57 (GND), J1.C58 (GND), J1.D03 (GND), J1.D06 (GND), J1.D09 (GND), J1.D12 (GND), J1.D15 (GND), J1.D19 (GND), J1.D23 (GND), J1.D27 (GND), J1.D31 (GND), J1.D35 (GND), J1.D39 (GND), J1.D43 (GND), J1.D47 (GND), J1.D48 (GND), J1.D51 (GND), J1.D52 (GND), J1.D55 (GND), J1.D56 (GND), J1.D59 (GND)
Other:
- moved on the sheet: H1, H2, H3, H4, H5, H6, H7, H8, J1A, J1B, J2A, J2B
