File: pcie_fpga/pcie_fpga.kicad_sch (KiCad schematic)
At the start: 26 parts, among them J1 PMOD_Host_Conn_02x06, J2 PCIexpress_x8, J3 PMOD_Host_Conn_02x06, J4 PMOD_Host_Conn_02x06, J5 87832-1420, U2 XCAU10P-1FFVB676I, X1 ECS-2520MVQ-1000-BN-TR

Commit message: pcie lanes need to be swapped I think.
Parts:
- added J6: Conn_02x03_Odd_Even, Connector_PinHeader_2.54mm:PinHeader_2x03_P2.54mm_Vertical, symbol Connector_Generic:Conn_02x03_Odd_Even
Connections:
- net prsntn: now also J6.2 (Pin_2), J6.4 (Pin_4), J6.6 (Pin_6); no longer J2.B48 (~{PRSNT2})
- net prsnt_x1: now reaches J2.B17 (~{PRSNT2})
- net prsnt_x1: now also J6.1 (Pin_1)
- net prsnt_x4: now reaches J2.B31 (~{PRSNT2})
- net prsnt_x4: now also J6.3 (Pin_3)
- new net prsnt_x8: J2.B48 (~{PRSNT2}), J6.5 (Pin_5)
Changed lines of the file:
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@@
   (junction (at 72.39 346.71) (diameter 0) (color 0 0 0 0)
   )
+  (junction (at 96.52 257.81) (diameter 0) (color 0 0 0 0)
+  )
   (junction (at 107.95 318.77) (diameter 0) (color 0 0 0 0)
   )
@@
   (junction (at 72.39 405.13) (diameter 0) (color 0 0 0 0)
   )
+  (junction (at 100.33 257.81) (diameter 0) (color 0 0 0 0)
+  )
   (junction (at 72.39 321.31) (diameter 0) (color 0 0 0 0)
   )
@@
   (junction (at 72.39 326.39) (diameter 0) (color 0 0 0 0)
   )
+  (junction (at 100.33 260.35) (diameter 0) (color 0 0 0 0)
+  )
   (junction (at 72.39 336.55) (diameter 0) (color 0 0 0 0)
   )
@@
     (stroke (width 0) (type default) (color 0 0 0 0))
   )
-  (wire (pts (xy 55.88 407.67) (xy 74.93 407.67))
-    (stroke (width 0) (type default) (color 0 0 0 0))
-  )
   (wire (pts (xy 105.41 387.35) (xy 127 387.35))
     (stroke (width 0) (type default) (color 0 0 0 0))
@@
     (stroke (width 0) (type default) (color 0 0 0 0))
   )
+  (wire (pts (xy 69.85 257.81) (xy 83.82 257.81))
+    (stroke (width 0) (type default) (color 0 0 0 0))
+  )
   (wire (pts (xy 74.93 339.09) (xy 72.39 339.09))
     (stroke (width 0) (type default) (color 0 0 0 0))
@@
     (stroke (width 0) (type default) (color 0 0 0 0))
   )
+  (wire (pts (xy 96.52 257.81) (xy 100.33 257.81))
+    (stroke (width 0) (type default) (color 0 0 0 0))
+  )
   (wire (pts (xy 74.93 364.49) (xy 72.39 364.49))
     (stroke (width 0) (type default) (color 0 0 0 0))
@@
     (stroke (width 0) (type default) (color 0 0 0 0))
   )
+  (wire (pts (xy 50.8 407.67) (xy 74.93 407.67))
+    (stroke (width 0) (type default) (color 0 0 0 0))
+  )
   (wire (pts (xy 105.41 407.67) (xy 127 407.67))
     (stroke (width 0) (type default) (color 0 0 0 0))
@@
     (stroke (width 0) (type default) (color 0 0 0 0))
   )
+  (wire (pts (xy 100.33 262.89) (xy 100.33 260.35))
+    (stroke (width 0) (type default) (color 0 0 0 0))
+  )
   (wire (pts (xy 107.95 278.13) (xy 107.95 283.21))
     (stroke (width 0) (type default) (color 0 0 0 0))
@@
     (stroke (width 0) (type default) (color 0 0 0 0))
   )
+  (wire (pts (xy 50.8 361.95) (xy 74.93 361.95))
+    (stroke (width 0) (type default) (color 0 0 0 0))
+  )
   (wire (pts (xy 287.02 340.36) (xy 308.61 340.36))
     (stroke (width 0) (type default) (color 0 0 0 0))
@@
     (stroke (width 0) (type default) (color 0 0 0 0))
   )
+  (wire (pts (xy 96.52 262.89) (xy 100.33 262.89))
+    (stroke (width 0) (type default) (color 0 0 0 0))
+  )
   (wire (pts (xy 72.39 414.02) (xy 72.39 410.21))
     (stroke (width 0) (type default) (color 0 0 0 0))
@@
     (stroke (width 0) (type default) (color 0 0 0 0))
   )
+  (wire (pts (xy 69.85 260.35) (xy 83.82 260.35))
+    (stroke (width 0) (type default) (color 0 0 0 0))
+  )
   (wire (pts (xy 69.85 298.45) (xy 74.93 298.45))
     (stroke (width 0) (type default) (color 0 0 0 0))
@@
     (stroke (width 0) (type default) (color 0 0 0 0))
   )
+  (wire (pts (xy 69.85 262.89) (xy 83.82 262.89))
+    (stroke (width 0) (type default) (color 0 0 0 0))
+  )
   (wire (pts (xy 72.39 326.39) (xy 72.39 321.31))
     (stroke (width 0) (type default) (color 0 0 0 0))
@@
     (stroke (width 0) (type default) (color 0 0 0 0))
   )
+  (wire (pts (xy 95.25 257.81) (xy 96.52 257.81))
+    (stroke (width 0) (type default) (color 0 0 0 0))
+  )
   (wire (pts (xy 455.93 346.71) (xy 455.93 344.17))
     (stroke (width 0) (type default) (color 0 0 0 0))
@@
     (stroke (width 0) (type default) (color 0 0 0 0))
   )
+  (wire (pts (xy 100.33 257.81) (xy 110.49 257.81))
+    (stroke (width 0) (type default) (color 0 0 0 0))
+  )
   (wire (pts (xy 163.83 403.86) (xy 185.42 403.86))
     (stroke (width 0) (type default) (color 0 0 0 0))
   )
+  (wire (pts (xy 100.33 260.35) (xy 100.33 257.81))
+    (stroke (width 0) (type default) (color 0 0 0 0))
+  )
   (wire (pts (xy 500.38 321.31) (xy 504.19 321.31))
     (stroke (width 0) (type default) (color 0 0 0 0))
@@
     (stroke (width 0) (type default) (color 0 0 0 0))
   )
+  (wire (pts (xy 96.52 260.35) (xy 100.33 260.35))
+    (stroke (width 0) (type default) (color 0 0 0 0))
+  )
   (wire (pts (xy 105.41 280.67) (xy 124.46 280.67))
     (stroke (width 0) (type default) (color 0 0 0 0))
@@
     (stroke (width 0) (type default) (color 0 0 0 0))
   )
+  (wire (pts (xy 50.8 323.85) (xy 74.93 323.85))
+    (stroke (width 0) (type default) (color 0 0 0 0))
+  )
   (wire (pts (xy 105.41 379.73) (xy 107.95 379.73))
     (stroke (width 0) (type default) (color 0 0 0 0))
@@
     (effects (font (size 1.27 1.27)) (justify left bottom))
   )
+  (label "prsnt_x4" (at 72.39 260.35 0)
+    (effects (font (size 1.27 1.27)) (justify left bottom))
+  )
   (label "per5_N" (at 143.51 388.62 0)
     (effects (font (size 1.27 1.27)) (justify left bottom))
@@
     (effects (font (size 1.27 1.27)) (justify left bottom))
   )
+  (label "prsnt_x8" (at 53.34 407.67 0)
+    (effects (font (size 1.27 1.27)) (justify left bottom))
+  )
   (label "pet4_P" (at 210.82 330.2 0)
     (effects (font (size 1.27 1.27)) (justify left bottom))
@@
     (effects (font (size 1.27 1.27)) (justify left bottom))
   )
+  (label "prsnt_x8" (at 72.39 262.89 0)
+    (effects (font (size 1.27 1.27)) (justify left bottom))
+  )
   (label "pre_per7_N" (at 170.18 408.94 0)
     (effects (font (size 1.27 1.27)) (justify left bottom))
@@
     (effects (font (size 1.27 1.27)) (justify left bottom))
   )
+  (label "prsnt_x4" (at 53.34 361.95 0)
+    (effects (font (size 1.27 1.27)) (justify left bottom))
+  )
+  (label "prsntn" (at 102.87 257.81 0)
+    (effects (font (size 1.27 1.27)) (justify left bottom))
+  )
   (label "ac_refclk_P" (at 170.18 303.53 0)
     (effects (font (size 1.27 1.27)) (justify left bottom))
@@
     (effects (font (size 1.27 1.27)) (justify left bottom))
   )
-  (label "prsntn" (at 59.69 407.67 0)
+  (label "per1_P" (at 111.76 336.55 0)
     (effects (font (size 1.27 1.27)) (justify left bottom))
   )
-  (label "per1_P" (at 111.76 336.55 0)
+  (label "prsnt_x1" (at 53.34 323.85 0)
     (effects (font (size 1.27 1.27)) (justify left bottom))
   )
@@
     (effects (font (size 1.27 1.27)) (justify left bottom))
   )
+  (label "prsnt_x1" (at 72.39 257.81 0)
+    (effects (font (size 1.27 1.27)) (justify left bottom))
+  )
   (label "pet2_P" (at 54.61 341.63 0)
     (effects (font (size 1.27 1.27)) (justify left bottom))
@@
     (pin "2")
   )
+  (symbol (lib_id "Connector_Generic:Conn_02x03_Odd_Even") (at 88.9 260.35 0) (unit 1)
+    (in_bom yes) (on_board yes) (fields_autoplaced)
+    (property "Reference" "J6" (id 0) (at 90.17 251.46 0))
+    (property "Value" "Conn_02x03_Odd_Even" (id 1) (at 90.17 254 0))
+    (property "Footprint" "Connector_PinHeader_2.54mm:PinHeader_2x03_P2.54mm_Vertical" (id 2) (at 88.9 260.35 0)
+      (effects (font (size 1.27 1.27)) hide)
+    )
+    (property "Datasheet" "~" (id 3) (at 88.9 260.35 0)
+      (effects (font (size 1.27 1.27)) hide)
+    )
+    (pin "1")
+    (pin "2")
+    (pin "3")
+    (pin "4")
+    (pin "5")
+    (pin "6")
+  )
   (symbol (lib_id "PCIexpress_x4_low-rescue:+3.3V-power") (at 69.85 298.45 90) (unit 1)
     (in_bom yes) (on_board yes)
@@
       (reference "J5") (unit 1) (value "87832-1420") (footprint "pedrolib:MOLEX_87832-1420")
     )
+    (path "/8733fca1-2e23-47d6-a6de-77f1b3f96389"
+      (reference "J6") (unit 1) (value "Conn_02x03_Odd_Even") (footprint "Connector_PinHeader_2.54mm:PinHeader_2x03_P2.54mm_Vertical")
+    )
     (path "/80450a8a-de64-4455-a65d-feef0126ac56"
