File: pcie/pcie_x1/PCIexpress_x1_low.kicad_pcb (KiCad board)
At the start: 4 copper layers, 167.7 x 68.9 mm, 3 parts, among them J1 PCIexpress_bracket, J2 PCIexpress_x1, U1 XC7A50T-FGG484

Commit message: working on x1 pcie card
Parts:
- added J2: PCIexpress_bracket, pedrolib:PCIexpress_bracket_low, F.Cu at (109.6, 194.1)
- added J3: PCIexpress_bracket, pedrolib:PCIexpress_bracket_low, F.Cu at (58.9, 69.0)
- renumbered J2 to J1
