File: custom_carrier/custom_carrier.kicad_sch (KiCad schematic)
At the start: 16 parts, among them J1 ERF5-040-05.0-X-DV, J13 PJ-002AH-SMT-TR, J14 87832-1420, J2 ERF5-040-05.0-X-DV, J3 ERF5-040-05.0-X-DV, J4 ERF5-040-05.0-X-DV, J5 45230-220230, J6 45230-220230

Commit message: added LED's
Parts:
- added D1, D2: LED, LED_SMD:LED_0603_1608Metric, symbol Device:LED
- added R4, R5: 240, Resistor_SMD:R_0603_1608Metric, symbol Device:R
Connections:
- net GND: now also D1.1 (K), D2.1 (K)
- net at J2.04: now also R4.1
- net at J2.34: now also R5.1
- new net: D1.2 (A), R4.2
- new net: D2.2 (A), R5.2
