File: mini_keyboard/kicad/mini_keyboard.kicad_sch (KiCad schematic)
At the start: 86 parts, among them U1 MX1A-11NN, U10 MX1A-11NN, U100 DEV-15583, U101 ABX00027, U11 MX1A-11NN, U12 MX1A-11NN, U13 MX1A-11NN, U14 MX1A-11NN, U15 MX1A-11NN, U16 MX1A-11NN, U17 MX1A-11NN, U18 MX1A-11NN, U19 MX1A-11NN, U2 MX1A-11NN, U20 MX1A-11NN, U21 MX1A-11NN, U22 MX1A-11NN, U23 MX1A-11NN, U24 MX1A-11NN, U25 MX1A-11NN, U26 MX1A-11NN, U27 MX1A-11NN, U28 MX1A-11NN, U29 MX1A-11NN, U3 MX1A-11NN, U30 MX1A-11NN, U31 MX1A-11NN, U32 MX1A-11NN, U33 MX1A-11NN, U34 MX1A-11NN, U35 MX1A-11NN, U36 MX1A-11NN, U37 MX1A-11NN, U38 MX1A-11NN, U39 MX1A-11NN, U4 MX1A-11NN, U40 MX1A-11NN, U41 MX1A-11NN, U42 MX1A-11NN, U5 MX1A-11NN, U6 MX1A-11NN, U7 MX1A-11NN, U8 MX1A-11NN, U9 MX1A-11NN

Commit message: looking at PG151101S11 socket for MX switches.
Parts:
- added S1: PG151101S11, pedrolib:SW_PG151101S11, symbol pedrolib:PG151101S11
Changed lines of the file:
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@@
+	)
+	(symbol
+		(lib_id "pedrolib:PG151101S11")
+		(at 54.61 186.69 0)
+		(unit 1)
+		(exclude_from_sim no)
+		(in_bom yes)
+		(on_board yes)
+		(dnp no)
+		(fields_autoplaced yes)
+		(property "Reference" "S1"
+			(at 54.61 179.07 0)
+			(effects
+				(font
+					(size 1.27 1.27)
+				)
+			)
+		)
+		(property "Value" "PG151101S11"
+			(at 54.61 181.61 0)
+			(effects
+				(font
+					(size 1.27 1.27)
+				)
+			)
+		)
+		(property "Footprint" "pedrolib:SW_PG151101S11"
+			(at 54.61 186.69 0)
+			(effects
+				(font
+					(size 1.27 1.27)
+				)
+				(justify bottom)
+				(hide yes)
+			)
+		)
+		(property "Datasheet" ""
+			(at 54.61 186.69 0)
+			(effects
+				(font
+					(size 1.27 1.27)
+				)
+				(hide yes)
+			)
+		)
+		(property "Description" ""
+			(at 54.61 186.69 0)
+			(effects
+				(font
+					(size 1.27 1.27)
+				)
+				(hide yes)
+			)
+		)
+		(property "MF" "Kailh"
+			(at 54.61 186.69 0)
+			(effects
+				(font
+					(size 1.27 1.27)
+				)
+				(justify bottom)
+				(hide yes)
+			)
+		)
+		(property "MAXIMUM_PACKAGE_HEIGHT" "1.95 mm"
+			(at 54.61 186.69 0)
+			(effects
+				(font
+					(size 1.27 1.27)
+				)
+				(justify bottom)
+				(hide yes)
+			)
+		)
+		(property "Package" "Package"
+			(at 54.61 186.69 0)
+			(effects
+				(font
+					(size 1.27 1.27)
+				)
+				(justify bottom)
+				(hide yes)
+			)
+		)
+		(property "Price" "None"
+			(at 54.61 186.69 0)
+			(effects
+				(font
+					(size 1.27 1.27)
+				)
+				(justify bottom)
+				(hide yes)
+			)
+		)
+		(property "Check_prices" "https://www.snapeda.com/parts/PG151101S11/Kailh/view-part/?ref=eda"
+			(at 54.61 186.69 0)
+			(effects
+				(font
+					(size 1.27 1.27)
+				)
+				(justify bottom)
+				(hide yes)
+			)
+		)
+		(property "STANDARD" "Manufacturer Recommendations"
+			(at 54.61 186.69 0)
+			(effects
+				(font
+					(size 1.27 1.27)
+				)
+				(justify bottom)
+				(hide yes)
+			)
+		)
+		(property "PARTREV" "A"
+			(at 54.61 186.69 0)
+			(effects
+				(font
+					(size 1.27 1.27)
+				)
+				(justify bottom)
+				(hide yes)
+			)
+		)
+		(property "SnapEDA_Link" "https://www.snapeda.com/parts/PG151101S11/Kailh/view-part/?ref=snap"
+			(at 54.61 186.69 0)
+			(effects
+				(font
+					(size 1.27 1.27)
+				)
+				(justify bottom)
+				(hide yes)
+			)
+		)
+		(property "MP" "PG151101S11"
+			(at 54.61 186.69 0)
+			(effects
+				(font
+					(size 1.27 1.27)
+				)
+				(justify bottom)
+				(hide yes)
+			)
+		)
+		(property "Description_1" "\n"
+			(at 54.61 186.69 0)
+			(effects
+				(font
+					(size 1.27 1.27)
+				)
+				(justify bottom)
+				(hide yes)
+			)
+		)
+		(property "Availability" "Not in stock"
+			(at 54.61 186.69 0)
+			(effects
+				(font
+					(size 1.27 1.27)
+				)
+				(justify bottom)
+				(hide yes)
+			)
+		)
+		(property "MANUFACTURER" "Kailh"
+			(at 54.61 186.69 0)
+			(effects
+				(font
+					(size 1.27 1.27)
+				)
+				(justify bottom)
+				(hide yes)
+			)
+		)
+		(pin "1"
+		)
+		(pin "2"
+		)
+		(instances
+			(project ""
+				(path "/25132092-e92d-469e-aa46-cb8dde2a6996"
+					(reference "S1")
+					(unit 1)
+				)
+			)
+		)
 	)
 	(symbol
